Commit message: Update vx300s.srdf.xacro

File: interbotix_ros_manipulators/interbotix_ros_xsarms/interbotix_xsarm_moveit/config/srdf/vx300s.srdf.xacro (robot description, xacro)
@@ -64,4 +64,8 @@
         <joint name="right_finger" value="-0.057" />
     </group_state>
+    <group_state name="Grasp_petridish" group="interbotix_gripper">
+        <joint name="left_finger" value="0.047" />
+        <joint name="right_finger" value="-0.047" />
+    </group_state>
     <group_state name="Home" group="interbotix_gripper">
         <joint name="left_finger" value="0.03" />

Commit message: Update vx300s.srdf.xacro

File: interbotix_ros_manipulators/interbotix_ros_xsarms/interbotix_xsarm_moveit/config/srdf/vx300s.srdf.xacro (robot description, xacro)
@@ -68,4 +68,8 @@
         <joint name="right_finger" value="-0.047" />
     </group_state>
+    <group_state name="Grasp_jelly" group="interbotix_gripper">
+        <joint name="left_finger" value="0.0185" />
+        <joint name="right_finger" value="-0.0185" />
+    </group_state>
     <group_state name="Home" group="interbotix_gripper">
         <joint name="left_finger" value="0.03" />
