Commit message: Update vx300s.urdf.xacro

File: interbotix_ros_manipulators/interbotix_ros_xsarms/interbotix_xsarm_descriptions/urdf/vx300s.urdf.xacro (robot description, xacro)
@@ -46,5 +46,5 @@
   <xacro:property name="gripper_limit_vel"          value="${pi}"/>
   <xacro:property name="finger_limit_effort"        value="5"/>
-  <xacro:property name="finger_limit_lower"         value="0.021"/>
+  <xacro:property name="finger_limit_lower"         value="0.017"/>
   <xacro:property name="finger_limit_upper"         value="0.057"/>
   <xacro:property name="finger_limit_vel"           value="1"/>

Commit message: Update vx300s.urdf.xacro

File: interbotix_ros_manipulators/interbotix_ros_xsarms/interbotix_xsarm_descriptions/urdf/vx300s.urdf.xacro (robot description, xacro)
@@ -97,4 +97,27 @@
     </inertial>
   </link>
+  <link name="camera_link">
+  <visual>
+     <origin
+        rpy="0 0 0"
+        xyz="0 0 0"/>
+      <geometry>
+        <box size="0.038 0.038 0.07" />
+      </geometry>
+      <material name="interbotix_black"/>
+  </visual>
+  </link>
+  <joint name="camera_joint" type="fixed">
+    <parent link="$(arg robot_name)/$(arg base_link_frame)" />
+    <child link="camera_link" />
+    <origin xyz="0.48 0.23 0.30" rpy="0 ${pi} 0" />
+  </joint>
+  <link name="camera_link_optical">
+  </link>
+  <joint name="camera_optical_joint" type="fixed">
+    <parent link="camera_link" />
+    <child link="camera_link_optical" />
+    <origin xyz="0 0 0" rpy="${-pi/2} 0 ${-pi/2}" />
+  </joint>
   <joint name="waist" type="revolute">
     <axis xyz="0 0 1"/>
